Commit message: latest

File: src/my_robot.urdf (robot description, URDF)
Before this commit: robot my_robot, 1 links, 0 joints
Links:
- added link lidar; visual cylinder length=0.2 radius=0.1
- link base_link: geometry visual box size=0.6 0.4 0.2
Joints:
- added joint base_lidar_joint: type fixed, parent base_link, child lidar, origin xyz=0 0 0 rpy=0 0 0
